File: brownies/circuits/hubcard/hubcard.kicad_pcb (KiCad board)
At the start: 2 copper layers, 99.1 x 83.8 mm, 12 parts, among them J1 Conn_02x10_Odd_Even, J2 Conn_02x04_Odd_Even, J3 Conn_01x03_Male, J4 Conn_01x04_Male, Q1 IRF5305, U1 ATtiny85V-10PU

Commit message: Add MQTT gateway driver; Add rain warning to weather driver; Improve floor plan UI; Many minor improvements
Parts:
- added D1: 6,8V, Diode_THT:D_DO-34_SOD68_P7.62mm_Horizontal, F.Cu at (45.7, 104.1)
- added D2: 6,8V, Diode_THT:D_DO-34_SOD68_P7.62mm_Horizontal, F.Cu at (43.2, 104.1)
- added D3: 6,8V, Diode_THT:D_DO-34_SOD68_P7.62mm_Horizontal, F.Cu at (58.4, 104.1)
Routing:
- net Net-(D1-Pad1): track 20.4 -> 35.6 mm
- net GND: track 203.3 -> 218.6 mm, vias 11 -> 12
- net Net-(D3-Pad1): track 12.7 -> 27.5 mm
- net Net-(D2-Pad1): track 10.2 -> 25.0 mm
